File: midicontroller8channels.sch (KiCad schematic (older format))
At the start: 71 parts, among them J1 Conn_01x02_Male, J10 Conn_01x02_Male, J11 Conn_01x02_Male, J12 Conn_01x02_Male, J13 Conn_01x12_Male, J14 Conn_01x12_Male, J15 Conn_01x12_Male, J16 Conn_01x12_Male, J17 Conn_01x03_Male, J18 Conn_01x08_Male, J19 Conn_01x04_Male, J2 Conn_01x02_Male, J3 Conn_01x02_Male, J4 Conn_01x02_Male, J5 Conn_01x12_Male, J6 Conn_01x12_Male, J7 Conn_01x12_Male, J8 Conn_01x12_Male, J9 Conn_01x02_Male, SW1 SW_Push, SW2 SW_Push, SW3 SW_Push, SW4 SW_Push, SW5 SW_Push, SW6 SW_Push, SW7 SW_Push, SW8 SW_Push, U1 4051, U2 4051, U3 4051, U4 4051

Commit message: vamooooo
Parts:
- removed J17: Conn_01x03_Male, Pin_Headers:Pin_Header_Straight_1x03_Pitch2.54mm, symbol Conn_01x03_Male
- removed J18: Conn_01x08_Male, Pin_Headers:Pin_Header_Straight_1x08_Pitch2.54mm, symbol Conn_01x08_Male
- added J17: Conn_01x05_Male, symbol Conn_01x05_Male
- added J18: Conn_01x06_Male, symbol Conn_01x06_Male
Connections:
- net D10: now also J17.3 (Pin_3)
- net D11: now also J17.2 (Pin_2)
- net D12: now also J17.1 (Pin_1)
- net D2: now also J18.6 (Pin_6)
- net D3: now also J18.5 (Pin_5)
- net D4: now also J18.4 (Pin_4)
- net D5: now also J18.3 (Pin_3)
- net D6: now also J18.2 (Pin_2)
- net D7: now also J18.1 (Pin_1)
- net D8: now also J17.5 (Pin_5)
- net D9: now also J17.4 (Pin_4)

Commit message: ay dios
Parts:
- J17: footprint (none) -> Pin_Headers:Pin_Header_Straight_1x05_Pitch2.54mm
- J18: footprint (none) -> Pin_Headers:Pin_Header_Straight_1x06_Pitch2.54mm

Commit message: finalizado
Parts:
- removed J13, J14, J15, J16, J5, J6, J7, J8: Conn_01x12_Male, Pin_Headers:Pin_Header_Straight_1x12_Pitch2.54mm, symbol Conn_01x12_Male
- removed J17: Conn_01x05_Male, Pin_Headers:Pin_Header_Straight_1x05_Pitch2.54mm, symbol Conn_01x05_Male
- removed J18: Conn_01x06_Male, Pin_Headers:Pin_Header_Straight_1x06_Pitch2.54mm, symbol Conn_01x06_Male
- removed J19: Conn_01x04_Male, Pin_Headers:Pin_Header_Straight_1x04_Pitch2.54mm, symbol Conn_01x04_Male
- added J10, J11, J12, J13, J14, J15, J16, J17, J18, J19, J20, J9: Conn_01x08_Male, Pin_Headers:Pin_Header_Straight_1x08_Pitch2.54mm, symbol Conn_01x08_Male
- added J21: arduinoUnoPinout, arduino:arduinoUnoPinout, symbol arduinoUnoPinout
- renumbered J9 to J5, J10 to J6, J11 to J7, J12 to J8
Connections:
- wire segments 349 -> 291
- no-connect marks 0 -> 12
