File: midicontroller8channels.kicad_pcb (KiCad board)
At the start: 2 copper layers, 86.4 x 73.7 mm, 33 parts, among them J1 Conn_01x02_Male, J10 Conn_01x08_Male, J11 Conn_01x08_Male, J12 Conn_01x08_Male, J13 Conn_01x08_Male, J14 Conn_01x08_Male, J15 Conn_01x08_Male, J16 Conn_01x08_Male, J17 Conn_01x08_Male, J18 Conn_01x08_Male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

Commit message: añado logo oshw
Parts:
- added REF***: OSHW-Logo2_7.3x6mm_SilkScreen, Symbols:OSHW-Logo2_7.3x6mm_SilkScreen, F.Cu at (154.9, 95.2)
Other:
- board text added: "20khzdesign juandarodriguez"
